Commit message: Simple IK from lerobot_kinematics

File: so101/so101.urdf (robot description, URDF)
Before this commit: robot so101, 8 links, 7 joints
Joints:
- joint wrist_roll: origin xyz=5.55112e-17 -0.0611 0.0181 rpy=1.5708 0.0486795 3.14159 -> xyz=5.55112e-17 -0.0611 0.0181 rpy=1.5708 0.0 3.14159
